Commit message: CKPT: working ver for shortcuts

File: src/pybullet_blocks/envs/broom.urdf (robot description, URDF)
Before this commit: robot broom, 2 links, 1 joints
Links:
- removed link base_link
- removed link base_link---short
- added link bristles, mass 0.05; collision box size=0.38 0.05 0.05; visual box size=0.38 0.05 0.05
- added link ferrule, mass 0.15; collision box size=0.4 0.06 0.02; visual box size=0.4 0.06 0.02
- added link handle, mass 0.1; collision box size=0.05 0.03 0.05; visual box size=0.1 0.03 0.05
Joints:
- removed joint hook_joint
- added joint ferrule_to_bristles: type fixed, parent ferrule, child bristles, origin xyz=0.0 0.0 -0.035 rpy=0 0 0
- added joint handle_to_ferrule: type fixed, parent handle, child ferrule, origin xyz=0.0 0.0 -0.01 rpy=0 0 0

Commit message: tune cleanuptable env

File: src/pybullet_blocks/envs/broom.urdf (robot description, URDF)
Before this commit: robot broom, 3 links, 2 joints
Links:
- link bristles: geometry collision box size=0.38 0.05 0.04; visual box size=0.38 0.05 0.04
Joints:
- joint ferrule_to_bristles: origin xyz=0.0 0.0 -0.035 rpy=0 0 0 -> xyz=0.0 0.0 -0.03 rpy=0 0 0
